Commit message: urdf file is launching in rviz properly

File: lidar_fuse_robot/urdf/robot_model.xacro (robot description, xacro)
@@ -27,77 +27,26 @@
         <parent link="base_link"/>
         <child link="chassis_1"/>
-        <origin xyz="0 0 0.135"/>
+        <origin xyz="0 0 0.11"/>
     </joint>
     <link name="chassis_1">
         <visual>
-            <origin xyz="0 0 0.0"/>
-            <geometry>
-                <box size="0.45 0.32 0.05"/>
-            </geometry>
-            <material name="silver"/>
-        </visual>
-        <collision>
-            <origin xyz="0 0 0.0"/>
-            <geometry>
-                <box size="0.45 0.32 0.05"/>
-            </geometry>
-        </collision>
-        <inertial>
-            <mass value="7.49"/>
-            <origin xyz="0 0 0"/>
-            <inertia ixx="0.0649" ixy="0" ixz="0" iyy="0.1433" iyz="0" izz="0.1926"/>
-        </inertial>
-    </link>
-    <joint name="chassis1_to_chassis2" type="fixed">
-        <parent link="chassis_1"/>
-        <child link="chassis_2"/>
-        <origin xyz="0 0 0.035"/>
-    </joint>
-    <link name="chassis_2">
-        <visual>
-            <origin xyz="0 0 0.0"/>
-            <geometry>
-                <box size="0.43 0.32 0.02"/>
+            <origin xyz="-0.325 -0.225 0.0"/>
+            <geometry>
+                <mesh filename="file://$(find lidar_fuse_robot)/stl/robot_base_top_plane.stl" scale="0.001 0.001 0.001"/>
             </geometry>
             <material name="white"/>
-            <gazebo reference="chassis_2">
-                <material>Gazebo/Orange</material>
-            </gazebo>
-        </visual>
-        <collision>
-            <origin xyz="0 0 0.0"/>
-            <geometry>
-                <box size="0.43 0.32 0.02"/>
-            </geometry>
-        </collision>
-        <inertial>
-            <mass value="2.86"/>
-            <origin xyz="0 0 0"/>
-            <inertia ixx="0.0244" ixy="0" ixz="0" iyy="0.0441" iyz="0" izz="0.0686"/>
-        </inertial>
-    </link>
-    <joint name="chassis2_to_chassis3" type="fixed">
-        <parent link="chassis_2"/>
-        <child link="chassis_3"/>
-        <origin xyz="0 0 0.03"/>
-    </joint>
-    <link name="chassis_3">
-        <visual>
-            <origin xyz="0 0 0.0"/>
-            <geometry>
-                <box size="0.45 0.32 0.04"/>
-            </geometry>
-            <material name="silver"/>
-        </visual>
-        <collision>
-            <origin xyz="0 0 0.0"/>
-            <geometry>
-                <box size="0.45 0.32 0.04"/>
-            </geometry>
-        </collision>
-        <inertial>
-            <mass value="5.99"/>
-            <origin xyz="0 0 0"/>
-            <inertia ixx="0.0517" ixy="0" ixz="0" iyy="0.1017" iyz="0" izz="0.1515"/>
+        </visual>
+        <collision>
+            <origin xyz="-0.325 -0.225 0.0"/>
+            <geometry>
+                <mesh filename="file://$(find lidar_fuse_robot)/stl/robot_base_top_plane.stl" scale="0.001 0.001 0.001"/>
+            </geometry>
+        </collision>
+        <inertial>
+            <mass value="23.62"/>
+            <origin xyz="-0.325 -0.225 0.0"/>
+            <inertia ixx="1.63" ixy="1.73" ixz="0.21"
+                    iyx="1.73" iyy="3.96" iyz="0.21"
+                    izx="0.21" izy="0.21" izz="4.89"/>
         </inertial>
     </link>
@@ -107,5 +56,5 @@
         <parent link="base_link"/>
         <child link="left_wheel"/>
-        <origin xyz="0.0 0.18 0.1" rpy="-${pi/2} 0.0 0.0"/>
+        <origin xyz="0.0 0.245 0.12" rpy="-${pi/2} 0.0 0.0"/>
         <axis xyz="0.0 0.0 1.0"/>
     </joint>
@@ -114,5 +63,5 @@
             <origin xyz="0.0 0.0 0.0"/>
             <geometry>
-                <cylinder radius="0.1" length="0.04"/>
+                <cylinder radius="0.12" length="0.04"/>
             </geometry>
             <material name="black"/>
@@ -121,5 +70,5 @@
             <origin xyz="0.0 0.0 0.0"/>
             <geometry>
-                <cylinder radius="0.1" length="0.04"/>
+                <cylinder radius="0.12" length="0.04"/>
             </geometry>
         </collision>
@@ -134,5 +83,5 @@
         <parent link="base_link"/>
         <child link="right_wheel"/>
-        <origin xyz="0.0 -0.18 0.1" rpy="${pi/2} 0.0 0.0"/>
+        <origin xyz="0.0 -0.245 0.12" rpy="${pi/2} 0.0 0.0"/>
         <axis xyz="0.0 0.0 -1.0"/>
     </joint>
@@ -141,5 +90,5 @@
             <origin xyz="0.0 0.0 0.0"/>
             <geometry>
-                <cylinder radius="0.1" length="0.04"/>
+                <cylinder radius="0.12" length="0.04"/>
             </geometry>
             <material name="black"/>
@@ -148,5 +97,5 @@
             <origin xyz="0.0 0.0 0.0"/>
             <geometry>
-                <cylinder radius="0.1" length="0.04"/>
+                <cylinder radius="0.12" length="0.04"/>
             </geometry>
         </collision>
@@ -159,7 +108,7 @@
     <!-- CASTER WHEEL LINK -->
     <joint name="caster_wheel_joint1" type="fixed">
-        <parent link="chassis_1"/>
+        <parent link="base_link"/>
         <child link="front_caster_wheel"/>
-        <origin xyz="0.145 0.0 -0.0675"/>
+        <origin xyz="0.20 -0.025 0.0"/>
         <axis xyz="0.0 0.0 0.0"/>
     </joint>
@@ -168,12 +117,12 @@
             <origin xyz="0.0 0.0 0.0"/>
             <geometry>
-                <sphere radius="0.0675"/>
-            </geometry>
-            <material name="grey"/>
-        </visual>
-        <collision>
-            <origin xyz="0.0 0.0 0.0"/>
-            <geometry>
-                <sphere radius="0.0675"/>
+                <mesh filename="file://$(find lidar_fuse_robot)/stl/caster_new_front_plane.stl" scale="0.001 0.001 0.001"/>
+            </geometry>
+            <material name="grey"/>
+        </visual>
+        <collision>
+            <origin xyz="0.0 0.0 0.0"/>
+            <geometry>
+                <mesh filename="file://$(find lidar_fuse_robot)/stl/caster_new_front_plane.stl" scale="0.001 0.001 0.001"/>
             </geometry>
             <material name="grey"/>
@@ -186,7 +135,7 @@
     </link>
     <joint name="caster_wheel_joint2" type="fixed">
-        <parent link="chassis_1"/>
+        <parent link="base_link"/>
         <child link="back_caster_wheel"/>
-        <origin xyz="-0.145 0.0 -0.0375"/>
+        <origin xyz="-0.25 -0.025 0.0"/>
         <axis xyz="0.0 0.0 0.0"/>
     </joint>
@@ -195,13 +144,14 @@
             <origin xyz="0.0 0.0 0.0"/>
             <geometry>
-                <sphere radius="0.0375"/>
-            </geometry>
-            <material name="grey"/>
-        </visual>
-        <collision>
-            <origin xyz="0.0 0.0 0.0"/>
-            <geometry>
-                <sphere radius="0.0375"/>
-            </geometry>
+                <mesh filename="file://$(find lidar_fuse_robot)/stl/caster_new_front_plane.stl" scale="0.001 0.001 0.001"/>
+            </geometry>
+            <material name="grey"/>
+        </visual>
+        <collision>
+            <origin xyz="0.0 0.0 0.0"/>
+            <geometry>
+                <mesh filename="file://$(find lidar_fuse_robot)/stl/caster_new_front_plane.stl" scale="0.001 0.001 0.001"/>
+            </geometry>
+            <material name="grey"/>
         </collision>
         <inertial>
@@ -211,7 +161,63 @@
         </inertial>
     </link>
-    <gazebo reference="chassis_2">
-        <material>Gazebo/Orange</material>
-    </gazebo>
+    <!--Lidar link-->
+    <joint name="front_lidar_joint" type="fixed">
+        <parent link="base_link"/>
+        <child link="front_lidar"/>
+        <origin xyz="0.24 0.140 0.075" rpy="0.0 0.0 -0.78"/>
+        <axis xyz="0.0 0.0 0.0"/>
+    </joint>
+        <link name="front_lidar">
+        <visual>
+            <origin xyz="-0.04 -0.02 -0.02"/>
+            <geometry>
+                <mesh filename="file://$(find lidar_fuse_robot)/stl/lidar_front.stl" scale="0.001 0.001 0.001"/>
+            </geometry>
+            <material name="blue"/>
+        </visual>
+        <collision>
+            <origin xyz="-0.04 -0.02 -0.02"/>
+            <geometry>
+                <mesh filename="file://$(find lidar_fuse_robot)/stl/lidar_front.stl" scale="0.001 0.001 0.001"/>
+            </geometry>
+            <material name="blue"/>
+        </collision>
+        <inertial>
+            <mass value="0.18"/>
+            <origin xyz="-0.04 -0.02 -0.02"/>
+            <inertia ixx="0.0009" ixy="-0.00032" ixz="0.00012"
+                    iyx="-0.00032" iyy="0.0010" iyz="-0.00028"
+                    izx="0.00012" izy="-0.00028" izz="0.00034"/>
+        </inertial>
+    </link>
+    <joint name="back_lidar_joint" type="fixed">
+        <parent link="base_link"/>
+        <child link="back_lidar"/>
+        <origin xyz="-0.24 -0.140 0.075" rpy="0.0 0.0 2.35619"/>
+        <axis xyz="0.0 0.0 0.0"/>
+    </joint>
+    <link name="back_lidar">
+        <visual>
+            <origin xyz="-0.04 -0.02 -0.02"/>
+            <geometry>
+                <mesh filename="file://$(find lidar_fuse_robot)/stl/lidar_front.stl" scale="0.001 0.001 0.001"/>
+            </geometry>
+            <material name="blue"/>
+        </visual>
+        <collision>
+            <origin xyz="-0.04 -0.02 -0.02"/>
+            <geometry>
+                <mesh filename="file://$(find lidar_fuse_robot)/stl/lidar_front.stl" scale="0.001 0.001 0.001"/>
+            </geometry>
+            <material name="blue"/>
+        </collision>
+        <inertial>
+            <mass value="0.18"/>
+            <origin xyz="-0.04 -0.02 -0.02"/>
+            <inertia ixx="0.0009" ixy="-0.00032" ixz="0.00012"
+                    iyx="-0.00032" iyy="0.0010" iyz="-0.00028"
+                    izx="0.00012" izy="-0.00028" izz="0.00034"/>
+        </inertial>
+    </link>
     <gazebo reference="left_wheel">
         <material>Gazebo/Blue</material>
