Commit message: Spawning the robot in Gazebo Classic
Spawning the robot with visualization turned on for both the lidars in gazebo classic

File: lidar_fuse_robot/urdf/lidar_bot.urdf.xacro (robot description, xacro)
@@ -2,3 +2,5 @@
 <robot xmlns:xacro = "http://www.ros.org/wiki/xacro" name="robot">
     <xacro:include filename="robot_model.xacro"/>
+    <xacro:include filename="gazebo_control.xacro"/>
+    <xacro:include filename="lidar.xacro"/>
 </robot>

File: lidar_fuse_robot/urdf/robot_model.xacro (robot description, xacro)
@@ -27,26 +27,83 @@
         <parent link="base_link"/>
         <child link="chassis_1"/>
-        <origin xyz="0 0 0.11"/>
+        <origin xyz="0 0 0.12"/>
     </joint>
     <link name="chassis_1">
         <visual>
-            <origin xyz="-0.325 -0.225 0.0"/>
-            <geometry>
-                <mesh filename="file://$(find lidar_fuse_robot)/stl/robot_base_top_plane.stl" scale="0.001 0.001 0.001"/>
+            <origin xyz="0 0 0.0"/>
+            <geometry>
+                <box size="0.60 0.40 0.05"/>
+            </geometry>
+            <material name="silver"/>
+        </visual>
+        <collision>
+            <origin xyz="0 0 0.0"/>
+            <geometry>
+                <box size="0.60 0.40 0.05"/>
+            </geometry>
+        </collision>
+        <inertial>
+            <origin xyz="0 0 0" rpy="0 0 0"/>
+            <mass value="12.48"/>
+            <inertia ixx="0.17" ixy="0.0" ixz="0.0"
+                    iyy="0.32" iyz="0.0"
+                    izz="0.47"/>
+        </inertial>
+    </link>
+    <joint name="chassis1_to_chassis2" type="fixed">
+        <parent link="chassis_1"/>
+        <child link="chassis_2"/>
+        <origin xyz="0 0 0.035"/>
+    </joint>
+    <link name="chassis_2">
+        <visual>
+            <origin xyz="0 0 0.0"/>
+            <geometry>
+                <box size="0.57 0.37 0.02"/>
             </geometry>
             <material name="white"/>
-        </visual>
-        <collision>
-            <origin xyz="-0.325 -0.225 0.0"/>
-            <geometry>
-                <mesh filename="file://$(find lidar_fuse_robot)/stl/robot_base_top_plane.stl" scale="0.001 0.001 0.001"/>
-            </geometry>
-        </collision>
-        <inertial>
-            <mass value="23.62"/>
-            <origin xyz="-0.325 -0.225 0.0"/>
-            <inertia ixx="1.63" ixy="1.73" ixz="0.21"
-                    iyx="1.73" iyy="3.96" iyz="0.21"
-                    izx="0.21" izy="0.21" izz="4.89"/>
+            <gazebo reference="chassis_2">
+                <material>Gazebo/Orange</material>
+            </gazebo>
+        </visual>
+        <collision>
+            <origin xyz="0 0 0.0"/>
+            <geometry>
+                <box size="0.57 0.37 0.02"/>
+            </geometry>
+        </collision>
+        <inertial>
+            <origin xyz="0 0 0" rpy="0 0 0"/>
+            <mass value="4.39"/>
+            <inertia ixx="0.04" ixy="0.0" ixz="0.0"
+                    iyy="0.10" iyz="0.0"
+                    izz="0.13"/>
+        </inertial>
+    </link>
+    <joint name="chassis2_to_chassis3" type="fixed">
+        <parent link="chassis_2"/>
+        <child link="chassis_3"/>
+        <origin xyz="0 0 0.03"/>
+    </joint>
+    <link name="chassis_3">
+        <visual>
+            <origin xyz="0 0 0.0"/>
+            <geometry>
+                <box size="0.60 0.40 0.04"/>
+            </geometry>
+            <material name="silver"/>
+        </visual>
+        <collision>
+            <origin xyz="0 0 0.0"/>
+            <geometry>
+                <box size="0.60 0.40 0.04"/>
+            </geometry>
+        </collision>
+        <inertial>
+            <origin xyz="0 0 0" rpy="0 0 0"/>
+            <mass value="9.98"/>
+            <inertia ixx="0.14" ixy="0.0" ixz="0.0"
+                    iyy="0.31" iyz="0.0"
+                    izz="0.41"/>
         </inertial>
     </link>
@@ -56,5 +113,5 @@
         <parent link="base_link"/>
         <child link="left_wheel"/>
-        <origin xyz="0.0 0.245 0.12" rpy="-${pi/2} 0.0 0.0"/>
+        <origin xyz="0.0 0.23 0.12" rpy="-${pi/2} 0.0 0.0"/>
         <axis xyz="0.0 0.0 1.0"/>
     </joint>
@@ -63,18 +120,20 @@
             <origin xyz="0.0 0.0 0.0"/>
             <geometry>
-                <cylinder radius="0.12" length="0.04"/>
-            </geometry>
-            <material name="black"/>
-        </visual>
-        <collision>
-            <origin xyz="0.0 0.0 0.0"/>
-            <geometry>
-                <cylinder radius="0.12" length="0.04"/>
-            </geometry>
-        </collision>
-        <inertial>
-            <mass value="1.06"/>
-            <origin xyz="0 0 0"/>
-            <inertia ixx="0.0026" ixy="0" ixz="0" iyy="0.0026" iyz="0" izz="0.00297"/>
+                <cylinder radius="0.12" length="0.06"/>
+            </geometry>
+            <material name="black"/>
+        </visual>
+        <collision>
+            <origin xyz="0.0 0.0 0.0"/>
+            <geometry>
+                <cylinder radius="0.12" length="0.06"/>
+            </geometry>
+        </collision>
+        <inertial>
+            <origin xyz="0 0 0" rpy="0 0 0"/>
+            <mass value="2.98"/>
+            <inertia ixx="0.0358" ixy="0.0" ixz="0.0"
+                    iyy="0.0358" iyz="0.0"
+                    izz="0.0214"/>
         </inertial>
     </link>
@@ -83,5 +142,5 @@
         <parent link="base_link"/>
         <child link="right_wheel"/>
-        <origin xyz="0.0 -0.245 0.12" rpy="${pi/2} 0.0 0.0"/>
+        <origin xyz="0.0 -0.23 0.12" rpy="${pi/2} 0.0 0.0"/>
         <axis xyz="0.0 0.0 -1.0"/>
     </joint>
@@ -90,136 +149,274 @@
             <origin xyz="0.0 0.0 0.0"/>
             <geometry>
-                <cylinder radius="0.12" length="0.04"/>
-            </geometry>
-            <material name="black"/>
-        </visual>
-        <collision>
-            <origin xyz="0.0 0.0 0.0"/>
-            <geometry>
-                <cylinder radius="0.12" length="0.04"/>
-            </geometry>
-        </collision>
-        <inertial>
-            <mass value="1.06"/>
-            <origin xyz="0 0 0"/>
-            <inertia ixx="0.0026" ixy="0" ixz="0" iyy="0.0026" iyz="0" izz="0.00297"/>
+                <cylinder radius="0.12" length="0.06"/>
+            </geometry>
+            <material name="black"/>
+        </visual>
+        <collision>
+            <origin xyz="0.0 0.0 0.0"/>
+            <geometry>
+                <cylinder radius="0.12" length="0.06"/>
+            </geometry>
+        </collision>
+        <inertial>
+            <origin xyz="0 0 0" rpy="0 0 0"/>
+            <mass value="2.98"/>
+            <inertia ixx="0.0358" ixy="0.0" ixz="0.0"
+                    iyy="0.0358" iyz="0.0"
+                    izz="0.0214"/>
         </inertial>
     </link>
     <!-- CASTER WHEEL LINK -->
-    <joint name="caster_wheel_joint1" type="fixed">
-        <parent link="base_link"/>
-        <child link="front_caster_wheel"/>
-        <origin xyz="0.20 -0.025 0.0"/>
+   <joint name="caster_wheel_joint1a" type="fixed">
+        <parent link="chassis_1"/>
+        <child link="front_caster_wheel_top"/>
+        <origin xyz="0.22 0.0 -0.05"/>
         <axis xyz="0.0 0.0 0.0"/>
     </joint>
-    <link name="front_caster_wheel">
-        <visual>
-            <origin xyz="0.0 0.0 0.0"/>
-            <geometry>
-                <mesh filename="file://$(find lidar_fuse_robot)/stl/caster_new_front_plane.stl" scale="0.001 0.001 0.001"/>
-            </geometry>
-            <material name="grey"/>
-        </visual>
-        <collision>
-            <origin xyz="0.0 0.0 0.0"/>
-            <geometry>
-                <mesh filename="file://$(find lidar_fuse_robot)/stl/caster_new_front_plane.stl" scale="0.001 0.001 0.001"/>
-            </geometry>
-            <material name="grey"/>
-        </collision>
-        <inertial>
-            <mass value="0.33"/>
-            <origin xyz="0 0 0"/>
-            <inertia ixx="0.00037" ixy="0" ixz="0" iyy="0.00037" iyz="0" izz="0.00037"/>
-        </inertial>
-    </link>
-    <joint name="caster_wheel_joint2" type="fixed">
-        <parent link="base_link"/>
-        <child link="back_caster_wheel"/>
-        <origin xyz="-0.25 -0.025 0.0"/>
+     <link name="front_caster_wheel_top">
+        <visual>
+            <origin xyz="0.0 0.0 0.0"/>
+            <geometry>
+                <box size="0.035 0.035 0.08"/>
+            </geometry>
+            <material name="white"/>
+        </visual>
+        <collision>
+            <origin xyz="0.0 0.0 0.0"/>
+            <geometry>
+                <box size="0.035 0.035 0.08"/>
+            </geometry>
+        </collision>
+        <inertial>
+            <origin xyz="0 0 0" rpy="0 0 0"/>
+            <mass value="0.102"/>
+            <inertia ixx="6.19e-5" ixy="0.0" ixz="0.0"
+                    iyy="6.19e-5" iyz="0.0"
+                    izz="2.70e-5"/>
+        </inertial>
+    </link>
+    <joint name="caster_wheel_joint1b" type="fixed">
+        <parent link="front_caster_wheel_top"/>
+        <child link="front_caster_wheel_bottom"/>
+        <origin xyz="0.0 0.0 -0.05"/>
         <axis xyz="0.0 0.0 0.0"/>
     </joint>
-    <link name="back_caster_wheel">
-        <visual>
-            <origin xyz="0.0 0.0 0.0"/>
-            <geometry>
-                <mesh filename="file://$(find lidar_fuse_robot)/stl/caster_new_front_plane.stl" scale="0.001 0.001 0.001"/>
-            </geometry>
-            <material name="grey"/>
-        </visual>
-        <collision>
-            <origin xyz="0.0 0.0 0.0"/>
-            <geometry>
-                <mesh filename="file://$(find lidar_fuse_robot)/stl/caster_new_front_plane.stl" scale="0.001 0.001 0.001"/>
-            </geometry>
-            <material name="grey"/>
-        </collision>
-        <inertial>
-            <mass value="0.33"/>
-            <origin xyz="0 0 0"/>
-            <inertia ixx="0.00037" ixy="0" ixz="0" iyy="0.00037" iyz="0" izz="0.00037"/>
-        </inertial>
-    </link>
-    <!--Lidar link-->
-    <joint name="front_lidar_joint" type="fixed">
-        <parent link="base_link"/>
+    <link name="front_caster_wheel_bottom">
+        <visual>
+            <origin xyz="0.0 0.0 0.0"/>
+            <geometry>
+                <sphere radius="0.02"/>
+            </geometry>
+            <material name="black"/>
+        </visual>
+        <collision>
+            <origin xyz="0.0 0.0 0.0"/>
+            <geometry>
+                <sphere radius="0.02"/>
+            </geometry>
+        </collision>
+        <inertial>
+            <origin xyz="0 0 0" rpy="0 0 0"/>
+            <mass value="0.0369"/>
+            <inertia ixx="2.95e-6" ixy="0.0" ixz="0.0"
+                    iyy="2.95e-6" iyz="0.0"
+                    izz="2.95e-6"/>
+        </inertial>
+    </link>
+    <joint name="caster_wheel_joint2a" type="fixed">
+        <parent link="chassis_1"/>
+        <child link="back_caster_wheel_top"/>
+        <origin xyz="-0.22 0.0 -0.05"/>
+        <axis xyz="0.0 0.0 0.0"/>
+    </joint>
+     <link name="back_caster_wheel_top">
+        <visual>
+            <origin xyz="0.0 0.0 0.0"/>
+            <geometry>
+                <box size="0.035 0.035 0.08"/>
+            </geometry>
+            <material name="white"/>
+        </visual>
+        <collision>
+            <origin xyz="0.0 0.0 0.0"/>
+            <geometry>
+                <box size="0.035 0.035 0.08"/>
+            </geometry>
+        </collision>
+        <inertial>
+            <origin xyz="0 0 0" rpy="0 0 0"/>
+            <mass value="0.102"/>
+            <inertia ixx="6.19e-5" ixy="0.0" ixz="0.0"
+                    iyy="6.19e-5" iyz="0.0"
+                    izz="2.70e-5"/>
+        </inertial>
+    </link>
+    <joint name="caster_wheel_joint2b" type="fixed">
+        <parent link="back_caster_wheel_top"/>
+        <child link="back_caster_wheel_bottom"/>
+        <origin xyz="0.0 0.0 -0.05"/>
+        <axis xyz="0.0 0.0 0.0"/>
+    </joint>
+    <link name="back_caster_wheel_bottom">
+        <visual>
+            <origin xyz="0.0 0.0 0.0"/>
+            <geometry>
+                <sphere radius="0.02"/>
+            </geometry>
+            <material name="black"/>
+        </visual>
+        <collision>
+            <origin xyz="0.0 0.0 0.0"/>
+            <geometry>
+                <sphere radius="0.02"/>
+            </geometry>
+        </collision>
+        <inertial>
+            <origin xyz="0 0 0" rpy="0 0 0"/>
+            <mass value="0.0369"/>
+            <inertia ixx="2.95e-6" ixy="0.0" ixz="0.0"
+                    iyy="2.95e-6" iyz="0.0"
+                    izz="2.95e-6"/>
+        </inertial>
+    </link>
+    <!-- Lidar Base Link -->
+    <joint name="chassis1_to_front_lidar_base" type="fixed">
+        <parent link="chassis_1"/>
+        <child link="front_lidar_base"/>
+        <origin xyz="0.25 0.15 -0.03"/>
+    </joint>
+    <link name="front_lidar_base">
+        <visual>
+            <origin xyz="0 0 0.0"/>
+            <geometry>
+                <box size="0.1 0.1 0.01"/>
+            </geometry>
+            <material name="black"/>
+        </visual>
+        <collision>
+            <origin xyz="0 0 0.0"/>
+            <geometry>
+                <box size="0.1 0.1 0.01"/>
+            </geometry>
+        </collision>
+        <inertial>
+            <origin xyz="0 0 0" rpy="0 0 0"/>
+            <mass value="0.104"/>
+            <inertia ixx="8.84e-5" ixy="0.0" ixz="0.0"
+                    iyy="8.84e-5" iyz="0.0"
+                    izz="1.77e-4"/>
+        </inertial>
+    </link>
+    <joint name="chassis1_to_back_lidar_base" type="fixed">
+        <parent link="chassis_1"/>
+        <child link="back_lidar_base"/>
+        <origin xyz="-0.25 -0.15 -0.03"/>
+    </joint>
+    <link name="back_lidar_base">
+        <visual>
+            <origin xyz="0 0 0.0"/>
+            <geometry>
+                <box size="0.1 0.1 0.01"/>
+            </geometry>
+            <material name="black"/>
+        </visual>
+        <collision>
+            <origin xyz="0 0 0.0"/>
+            <geometry>
+                <box size="0.1 0.1 0.01"/>
+            </geometry>
+        </collision>
+        <inertial>
+            <origin xyz="0 0 0" rpy="0 0 0"/>
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