Commit message: UPDATE - code is workinggit add .git add .git add .git add .git add .git add .git add .git add .git add .

File: lidar_fuse_robot/urdf/lidar.xacro (robot description, xacro)
@@ -10,6 +10,6 @@
                         <horizontal>
                             <samples>360</samples>
-                            <min_angle>4.64</min_angle>
-                            <max_angle>8.74</max_angle>
+                            <min_angle>-1.60</min_angle>
+                            <max_angle>2.45</max_angle>
                         </horizontal>
                     </scan>
@@ -37,6 +37,6 @@
                         <horizontal>
                             <samples>360</samples>
-                            <min_angle>1.51</min_angle>
-                            <max_angle>5.59</max_angle>
+                            <min_angle>-1.60</min_angle>
+                            <max_angle>2.45</max_angle>
                         </horizontal>
                     </scan>

File: lidar_fuse_robot/urdf/robot_model.xacro (robot description, xacro)
@@ -336,7 +336,7 @@
     </link>
     <joint name="front_lidar_base_to_front_lidar" type="fixed">
-        <parent link="front_lidar_base"/>
+        <parent link="base_link"/>
         <child link="front_lidar"/>
-        <origin xyz="0.00 0.00 -0.02"/>
+        <origin xyz="0.25 0.15 0.07"/>
     </joint>
     <link name="front_lidar">
@@ -363,7 +363,7 @@
     </link>
     <joint name="back_lidar_base_to_back_lidar" type="fixed">
-        <parent link="back_lidar_base"/>
+        <parent link="base_link"/>
         <child link="back_lidar"/>
-        <origin xyz="0.00 0.00 -0.02"/>
+        <origin xyz="-0.25 -0.15 0.07" rpy = "0.0 0.0 ${pi}"/>
     </joint>
     <link name="back_lidar">
